File: hardware/v1.1-RH/elektronika.kicad_sch (KiCad schematic)
At the start: 50 parts, among them J2 Conn_01x06_Male, J3 USB_C_Receptacle_USB2.0, J8 Conn_01x10_Male, Q1 Q_NPN_BEC, Q2 Q_NPN_BEC, Q4 Q_NMOS_GSD, Q5 Q_PMOS_GSD, Q6 Q_NMOS_GSD, Q7 Q_NMOS_GSD, Q8 Q_NMOS_GSD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

Commit message: Final touch for the RH version
Parts:
- removed DRA2: Logo_Robotarna, my_library:RobotarnaLogo-6mm, symbol Mechanical:DIN_Rail_Adapter
Changed lines of the file:
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@@
     (pin "3")
-  )
-  (symbol (lib_id "Mechanical:DIN_Rail_Adapter") (at 72.39 187.96 0) (unit 1)
-    (in_bom yes) (on_board yes)
-    (property "Reference" "DRA2" (id 0) (at 72.39 181.229 0))
-    (property "Value" "Logo_Robotarna" (id 1) (at 72.39 183.5404 0))
-    (property "Footprint" "my_library:RobotarnaLogo-6mm" (id 2) (at 72.39 193.04 0)
-      (effects (font (size 1.27 1.27)) hide)
-    )
-    (property "Datasheet" "~" (id 3) (at 72.39 184.15 0)
-      (effects (font (size 1.27 1.27)) hide)
-    )
-    (property "LCSC" "-" (id 4) (at 72.39 187.96 0)
-      (effects (font (size 1.27 1.27)) hide)
-    )
-    (property "JLCPCB_CORRECTION" "0;0;0" (id 5) (at 72.39 187.96 0)
-      (effects (font (size 1.27 1.27)) hide)
-    )
   )
   (symbol (lib_id "Device:R") (at 64.77 91.44 0) (unit 1)
