File: hardware/v1.1-RH/LEDky5.kicad_sch (KiCad schematic)
At the start: 10 parts

Commit message: Fix LED correction
Parts:
- D12, D13, D14, D15, D16: JLCPCB_CORRECTION 0;0;180 -> 0;0;0
Changed lines of the file:
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@@
       (effects (font (size 1.27 1.27)) hide)
     )
-    (property "JLCPCB_CORRECTION" "0;0;180" (id 5) (at 71.12 92.71 0)
+    (property "JLCPCB_CORRECTION" "0;0;0" (id 5) (at 71.12 92.71 0)
       (effects (font (size 1.27 1.27)) hide)
     )
@@
       (effects (font (size 1.27 1.27)) hide)
     )
-    (property "JLCPCB_CORRECTION" "0;0;180" (id 5) (at 106.68 92.71 0)
+    (property "JLCPCB_CORRECTION" "0;0;0" (id 5) (at 106.68 92.71 0)
       (effects (font (size 1.27 1.27)) hide)
     )
@@
       (effects (font (size 1.27 1.27)) hide)
     )
-    (property "JLCPCB_CORRECTION" "0;0;180" (id 5) (at 139.7 92.71 0)
+    (property "JLCPCB_CORRECTION" "0;0;0" (id 5) (at 139.7 92.71 0)
       (effects (font (size 1.27 1.27)) hide)
     )
@@
       (effects (font (size 1.27 1.27)) hide)
     )
-    (property "JLCPCB_CORRECTION" "0;0;180" (id 5) (at 175.26 92.71 0)
+    (property "JLCPCB_CORRECTION" "0;0;0" (id 5) (at 175.26 92.71 0)
       (effects (font (size 1.27 1.27)) hide)
     )
@@
       (effects (font (size 1.27 1.27)) hide)
     )
-    (property "JLCPCB_CORRECTION" "0;0;180" (id 5) (at 207.01 92.71 0)
+    (property "JLCPCB_CORRECTION" "0;0;0" (id 5) (at 207.01 92.71 0)
       (effects (font (size 1.27 1.27)) hide)
     )
