File: hardware/v1.1-RH/zadani_LED.kicad_sch (KiCad schematic)
At the start: 10 parts

Commit message: Fix LED correction
Parts:
- D113, D3, D4, D5, D6: JLCPCB_CORRECTION 0;0;180 -> 0;0;0
Changed lines of the file:
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@@
       (effects (font (size 1.27 1.27)) hide)
     )
-    (property "JLCPCB_CORRECTION" "0;0;180" (id 5) (at 97.79 96.52 0)
+    (property "JLCPCB_CORRECTION" "0;0;0" (id 5) (at 97.79 96.52 0)
       (effects (font (size 1.27 1.27)) hide)
     )
@@
       (effects (font (size 1.27 1.27)) hide)
     )
-    (property "JLCPCB_CORRECTION" "0;0;180" (id 5) (at 130.81 96.52 0)
+    (property "JLCPCB_CORRECTION" "0;0;0" (id 5) (at 130.81 96.52 0)
       (effects (font (size 1.27 1.27)) hide)
     )
@@
       (effects (font (size 1.27 1.27)) hide)
     )
-    (property "JLCPCB_CORRECTION" "0;0;180" (id 5) (at 166.37 96.52 0)
+    (property "JLCPCB_CORRECTION" "0;0;0" (id 5) (at 166.37 96.52 0)
       (effects (font (size 1.27 1.27)) hide)
     )
@@
       (effects (font (size 1.27 1.27)) hide)
     )
-    (property "JLCPCB_CORRECTION" "0;0;180" (id 5) (at 199.39 96.52 0)
+    (property "JLCPCB_CORRECTION" "0;0;0" (id 5) (at 199.39 96.52 0)
       (effects (font (size 1.27 1.27)) hide)
     )
@@
       (effects (font (size 1.27 1.27)) hide)
     )
-    (property "JLCPCB_CORRECTION" "0;0;180" (id 5) (at 227.33 96.52 0)
+    (property "JLCPCB_CORRECTION" "0;0;0" (id 5) (at 227.33 96.52 0)
       (effects (font (size 1.27 1.27)) hide)
     )
