File: hardware/v2.0/ovladaci_prvky.kicad_sch (KiCad schematic)
At the start: 8 parts, among them Q3 Q_Photo_NPN

Commit message: Secondary button cross
Other:
- sheet tlacitka.sch ports: added SW_12; removed none
Changed lines of the file:
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@@
+    (stroke (width 0) (type default) (color 0 0 0 0))
+  )
+  (wire (pts (xy 119.38 99.06) (xy 114.3 99.06))
     (stroke (width 0) (type default) (color 0 0 0 0))
   )
@@
   (hierarchical_label "GND" (shape input) (at 207.01 64.77 270)
     (effects (font (size 1.27 1.27)) (justify right))
+  )
+  (hierarchical_label "SW_12" (shape input) (at 119.38 99.06 0)
+    (effects (font (size 1.27 1.27)) (justify left))
   )
   (hierarchical_label "SW_9" (shape input) (at 119.38 85.09 0)
@@
       (effects (font (size 1.27 1.27)) (justify right))
     )
+    (pin "SW_12" input (at 114.3 99.06 0)
+      (effects (font (size 1.27 1.27)) (justify right))
+    )

Commit message: Change piezo
Parts:
- Q3: JLCPCB_CORRECTION 0;0;0 -> 0;0;180
Changed lines of the file:
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@@
       (effects (font (size 1.27 1.27)) hide)
     )
-    (property "JLCPCB_CORRECTION" "0;0;0" (id 4) (at 251.46 78.74 0)
+    (property "JLCPCB_CORRECTION" "0;0;180" (id 4) (at 251.46 78.74 0)
       (effects (font (size 1.27 1.27)) hide)
     )
