File: hardware/v2.0/tlacitka.kicad_sch (KiCad schematic)
At the start: 18 parts, among them SW10 button, SW11 button, SW2 button, SW3 button, SW4 button, SW5 button, SW7 button, SW8 button, SW9 button

Commit message: Secondary button cross
Parts:
- added C30: 10n, Capacitor_SMD:C_0402_1005Metric, symbol Device:C
- added SW12: button, my_library:Tactile_switch, symbol Switch:SW_Push
Connections:
- net GND: now also C30.1, SW12.2
- new net SW_12: C30.2, SW12.1
Changed lines of the file:
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@@
   (junction (at 168.91 110.49) (diameter 0) (color 0 0 0 0)
   )
+  (junction (at 168.91 130.81) (diameter 0) (color 0 0 0 0)
+  )
   (junction (at 130.81 40.64) (diameter 0) (color 0 0 0 0)
   )
@@
   (junction (at 186.69 82.55) (diameter 0) (color 0 0 0 0)
   )
+  (junction (at 186.69 130.81) (diameter 0) (color 0 0 0 0)
+  )
   (junction (at 168.91 40.64) (diameter 0) (color 0 0 0 0)
   )
@@
     (stroke (width 0) (type default) (color 0 0 0 0))
   )
+  (wire (pts (xy 172.72 130.81) (xy 168.91 130.81))
+    (stroke (width 0) (type default) (color 0 0 0 0))
+  )
   (wire (pts (xy 135.89 60.96) (xy 130.81 60.96))
     (stroke (width 0) (type default) (color 0 0 0 0))
@@
     (stroke (width 0) (type default) (color 0 0 0 0))
   )
+  (wire (pts (xy 182.88 130.81) (xy 186.69 130.81))
+    (stroke (width 0) (type default) (color 0 0 0 0))
+  )
   (wire (pts (xy 186.69 110.49) (xy 186.69 115.57))
     (stroke (width 0) (type default) (color 0 0 0 0))
@@
     (stroke (width 0) (type default) (color 0 0 0 0))
   )
+  (wire (pts (xy 168.91 135.89) (xy 173.99 135.89))
+    (stroke (width 0) (type default) (color 0 0 0 0))
+  )
   (wire (pts (xy 113.03 135.89) (xy 118.11 135.89))
     (stroke (width 0) (type default) (color 0 0 0 0))
@@
     (stroke (width 0) (type default) (color 0 0 0 0))
   )
+  (wire (pts (xy 165.1 130.81) (xy 168.91 130.81))
+    (stroke (width 0) (type default) (color 0 0 0 0))
+  )
   (wire (pts (xy 191.77 60.96) (xy 186.69 60.96))
     (stroke (width 0) (type default) (color 0 0 0 0))
@@
     (stroke (width 0) (type default) (color 0 0 0 0))
   )
+  (wire (pts (xy 191.77 130.81) (xy 186.69 130.81))
+    (stroke (width 0) (type default) (color 0 0 0 0))
+  )
   (wire (pts (xy 110.49 82.55) (xy 114.3 82.55))
     (stroke (width 0) (type default) (color 0 0 0 0))
   )
+  (wire (pts (xy 168.91 130.81) (xy 168.91 135.89))
+    (stroke (width 0) (type default) (color 0 0 0 0))
+  )
   (wire (pts (xy 127 110.49) (xy 130.81 110.49))
     (stroke (width 0) (type default) (color 0 0 0 0))
@@
     (stroke (width 0) (type default) (color 0 0 0 0))
   )
+  (wire (pts (xy 186.69 135.89) (xy 181.61 135.89))
+    (stroke (width 0) (type default) (color 0 0 0 0))
+  )
   (wire (pts (xy 165.1 40.64) (xy 168.91 40.64))
     (stroke (width 0) (type default) (color 0 0 0 0))
@@
     (stroke (width 0) (type default) (color 0 0 0 0))
   )
+  (wire (pts (xy 186.69 130.81) (xy 186.69 135.89))
+    (stroke (width 0) (type default) (color 0 0 0 0))
+  )
   (wire (pts (xy 116.84 40.64) (xy 113.03 40.64))
     (stroke (width 0) (type default) (color 0 0 0 0))
@@
     (effects (font (size 1.27 1.27)) (justify left))
   )
+  (hierarchical_label "SW_12" (shape input) (at 165.1 130.81 180)
+    (effects (font (size 1.27 1.27)) (justify right))
+  )
   (hierarchical_label "SW_2" (shape input) (at 109.22 40.64 180)
     (effects (font (size 1.27 1.27)) (justify right))
@@
   (hierarchical_label "SW_10" (shape input) (at 165.1 82.55 180)
     (effects (font (size 1.27 1.27)) (justify right))
+  )
+  (hierarchical_label "GND" (shape input) (at 191.77 130.81 0)
+    (effects (font (size 1.27 1.27)) (justify left))
   )
   (hierarchical_label "SW_11" (shape input) (at 165.1 110.49 180)
@@
       (effects (font (size 1.27 1.27)) hide)
     )
+    (pin "1")
+    (pin "2")
+  )
+  (symbol (lib_id "Device:C") (at 177.8 135.89 270) (unit 1)
+    (in_bom yes) (on_board yes)
+    (property "Reference" "C30" (id 0) (at 181.61 137.16 90))
+    (property "Value" "10n" (id 1) (at 177.8 131.8006 90))
+    (property "Footprint" "Capacitor_SMD:C_0402_1005Metric" (id 2) (at 173.99 136.8552 0)
+      (effects (font (size 1.27 1.27)) hide)
+    )
+    (property "Datasheet" "~" (id 3) (at 177.8 135.89 0)
+      (effects (font (size 1.27 1.27)) hide)
+    )
+    (property "LCSC" "C15195" (id 4) (at 177.8 135.89 0)
+      (effects (font (size 1.27 1.27)) hide)
+    )
+    (property "JLCPCB_CORRECTION" "0;0;0" (id 5) (at 177.8 135.89 0)
+      (effects (font (size 1.27 1.27)) hide)
+    )
+    (pin "1")
+    (pin "2")
+  )
+  (symbol (lib_id "Switch:SW_Push") (at 177.8 130.81 0) (unit 1)
+    (in_bom yes) (on_board yes)
+    (property "Reference" "SW12" (id 0) (at 177.8 123.571 0))
+    (property "Value" "button" (id 1) (at 177.8 125.8824 0))
+    (property "Footprint" "my_library:Tactile_switch" (id 2) (at 177.8 125.73 0)
+      (effects (font (size 1.27 1.27)) hide)
+    )
+    (property "Datasheet" "~" (id 3) (at 177.8 125.73 0)
+      (effects (font (size 1.27 1.27)) hide)
+    )
+    (property "LCSC" "C318887" (id 4) (at 177.8 130.81 0)
+      (effects (font (size 1.27 1.27)) hide)
+    )
+    (property "JLCPCB_CORRECTION" "0;0;0" (id 5) (at 177.8 130.81 0)
+      (effects (font (size 1.27 1.27)) hide)
+    )
