File: hardware/v2.0/Logic_tabor.kicad_sch (KiCad schematic)
At the start: 8 parts, among them J10 Conn_01x04_Male, J4 Conn_01x07_Female, J5 Conn_01x04_Female, J6 Conn_01x04_Female, J7 Conn_01x07_Male, J9 Conn_01x04_Male

Commit message: Secondary button cross
Parts:
- removed J10, J9: Conn_01x04_Male, Connector_PinHeader_2.54mm:PinHeader_1x04_P2.54mm_Vertical, symbol Connector:Conn_01x04_Male
- removed J4: Conn_01x07_Female, Connector_PinHeader_2.54mm:PinHeader_1x07_P2.54mm_Vertical, symbol Connector:Conn_01x07_Female
- removed J5, J6: Conn_01x04_Female, Connector_PinHeader_2.54mm:PinHeader_1x04_P2.54mm_Vertical, symbol Connector:Conn_01x04_Female
- removed J7: Conn_01x07_Male, Connector_PinHeader_2.54mm:PinHeader_1x07_P2.54mm_Vertical, symbol Connector:Conn_01x07_Male
- added J10, J5, J6, J9: Conn_01x04, Connector_PinHeader_2.54mm:PinHeader_1x04_P2.54mm_Vertical, symbol Connector_Generic:Conn_01x04
- added J4, J7: Conn_01x08, Connector_PinSocket_2.54mm:PinSocket_1x08_P2.54mm_Vertical, symbol Connector_Generic:Conn_01x08
Connections:
- net elektronika.sch/3V3: now also J7.1 (Pin_1)
- net elektronika.sch/DATA_HERNI_LED: now also J7.5 (Pin_5)
- net elektronika.sch/DATA_ZADANI_LED: now also J7.4 (Pin_4)
- net elektronika.sch/GND: now also J7.3 (Pin_3)
- net elektronika.sch/SENZOR_SVETLA: now also J7.7 (Pin_7)
- net elektronika.sch/SW_10: now also J9.3 (Pin_3)
- net elektronika.sch/SW_11: now also J10.1 (Pin_1)
- net elektronika.sch/SW_2: now also J10.4 (Pin_4)
- net elektronika.sch/SW_3: now also J10.3 (Pin_3)
- net elektronika.sch/SW_4: now also J9.4 (Pin_4)
- net elektronika.sch/SW_5: now also J9.1 (Pin_1)
- net elektronika.sch/SW_7: now also J7.2 (Pin_2)
- net elektronika.sch/SW_8: now also J10.2 (Pin_2)
- net elektronika.sch/SW_9: now also J9.2 (Pin_2)
- net elektronika.sch/V_LED_1: now also J7.6 (Pin_6)
- net ovladaci_prvky.sch/3V3: now also J4.1 (Pin_1)
- net ovladaci_prvky.sch/DATA_HERNI_LED: now also J4.5 (Pin_5)
- net ovladaci_prvky.sch/DATA_ZADANI_LED: now also J4.4 (Pin_4)
- net ovladaci_prvky.sch/GND: now also J4.3 (Pin_3)
- net ovladaci_prvky.sch/SENZOR_SVETLA: now also J4.7 (Pin_7)
- net ovladaci_prvky.sch/SW_10: now also J5.3 (Pin_3)
- net ovladaci_prvky.sch/SW_11: now also J6.1 (Pin_1)
- net ovladaci_prvky.sch/SW_2: now also J6.4 (Pin_4)
- net ovladaci_prvky.sch/SW_3: now also J6.3 (Pin_3)
- net ovladaci_prvky.sch/SW_4: now also J5.4 (Pin_4)
- net ovladaci_prvky.sch/SW_5: now also J5.1 (Pin_1)
- net ovladaci_prvky.sch/SW_7: now also J4.2 (Pin_2)
- net ovladaci_prvky.sch/SW_8: now also J6.2 (Pin_2)
- net ovladaci_prvky.sch/SW_9: now also J5.2 (Pin_2)
- net ovladaci_prvky.sch/V_LED_1: now also J4.6 (Pin_6)
- new net elektronika.sch/SW_12: J7.8 (Pin_8)
- new net ovladaci_prvky.sch/SW_12: J4.8 (Pin_8)
Other:
- sheet elektronika.sch ports: added SW_12; removed none
- sheet ovladaci_prvky.sch ports: added SW_12; removed none

Commit message: SD karta and factory files
Parts:
- J5, J6: footprint Connector_PinHeader_2.54mm:PinHeader_1x04_P2.54mm_Vertical -> Connector_PinSocket_2.54mm:PinSocket_1x04_P2.54mm_Vertical
- J7: footprint Connector_PinSocket_2.54mm:PinSocket_1x08_P2.54mm_Vertical -> Connector_PinHeader_2.54mm:PinHeader_1x08_P2.54mm_Vertical
Changed lines of the file:
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@@
     (property "Reference" "J7" (id 0) (at 160.02 68.58 0))
     (property "Value" "Conn_01x08" (id 1) (at 160.02 71.12 0))
-    (property "Footprint" "Connector_PinSocket_2.54mm:PinSocket_1x08_P2.54mm_Vertical" (id 2) (at 160.02 81.28 0)
+    (property "Footprint" "Connector_PinHeader_2.54mm:PinHeader_1x08_P2.54mm_Vertical" (id 2) (at 160.02 81.28 0)
       (effects (font (size 1.27 1.27)) hide)
     )
@@
       (effects (font (size 1.27 1.27)) (justify left))
     )
-    (property "Footprint" "Connector_PinHeader_2.54mm:PinHeader_1x04_P2.54mm_Vertical" (id 2) (at 144.78 111.76 0)
+    (property "Footprint" "Connector_PinSocket_2.54mm:PinSocket_1x04_P2.54mm_Vertical" (id 2) (at 144.78 111.76 0)
       (effects (font (size 1.27 1.27)) hide)
     )
@@
       (effects (font (size 1.27 1.27)) (justify left))
     )
-    (property "Footprint" "Connector_PinHeader_2.54mm:PinHeader_1x04_P2.54mm_Vertical" (id 2) (at 144.78 101.6 0)
+    (property "Footprint" "Connector_PinSocket_2.54mm:PinSocket_1x04_P2.54mm_Vertical" (id 2) (at 144.78 101.6 0)
       (effects (font (size 1.27 1.27)) hide)
     )
@@
       (reference "C21") (unit 1) (value "100n") (footprint "Capacitor_SMD:C_0402_1005Metric")
     )
-    (path "/00000000-0000-0000-0000-00006025abb3/af17f6b3-11fc-4bbd-aba0-f73fb0159317/e77a964e-09a0-46ee-88d4-c9c46170195b"
-      (reference "C22") (unit 1) (value "10u") (footprint "Capacitor_SMD:C_0402_1005Metric")
-    )
-    (path "/00000000-0000-0000-0000-00006025abb3/af17f6b3-11fc-4bbd-aba0-f73fb0159317/00cf874a-22ca-44ec-acb3-f2ecb134a5a6"
-      (reference "C23") (unit 1) (value "10u") (footprint "Capacitor_SMD:C_0402_1005Metric")
-    )
-    (path "/00000000-0000-0000-0000-00006025abb3/af17f6b3-11fc-4bbd-aba0-f73fb0159317/73fab6f8-d9a7-4b38-b41b-3c71c67fe103"
-      (reference "C24") (unit 1) (value "10u") (footprint "Capacitor_SMD:C_0402_1005Metric")
+    (path "/00000000-0000-0000-0000-00006025abb3/be53324f-912d-402f-9c60-3bf81cba9d8e"
+      (reference "C22") (unit 1) (value "10uF") (footprint "Capacitor_SMD:C_0603_1608Metric")
+    )
+    (path "/00000000-0000-0000-0000-00006025abb3/8e2c2a0a-a1e0-4221-abc1-5b757109c53d"
+      (reference "C23") (unit 1) (value "10uF") (footprint "Capacitor_SMD:C_0603_1608Metric")
+    )
+    (path "/00000000-0000-0000-0000-00006025abb3/af17f6b3-11fc-4bbd-aba0-f73fb0159317/8f43f925-c85b-4f98-9d39-4d325523de71"
+      (reference "C24") (unit 1) (value "10uF") (footprint "Capacitor_SMD:C_0603_1608Metric")
     )
     (path "/00000000-0000-0000-0000-00006025abb3/af17f6b3-11fc-4bbd-aba0-f73fb0159317/42c814c2-1ccf-48ba-8371-cc70437d09ca"
@@
     )
     (path "/00000000-0000-0000-0000-00006025abb3/af17f6b3-11fc-4bbd-aba0-f73fb0159317/ae05f26a-f12a-42fb-a09b-79b1f5107ac8"
-      (reference "C27") (unit 1) (value "10u") (footprint "Capacitor_SMD:C_0402_1005Metric")
+      (reference "C27") (unit 1) (value "10uF") (footprint "Capacitor_SMD:C_0603_1608Metric")
     )
     (path "/00000000-0000-0000-0000-00006025abb3/af17f6b3-11fc-4bbd-aba0-f73fb0159317/a673fa3b-d490-4d62-bca2-2ad44d46987b"
@@
       (reference "C126") (unit 1) (value "10n") (footprint "Capacitor_SMD:C_0402_1005Metric")
     )
+    (path "/00000000-0000-0000-0000-00006025abb3/af17f6b3-11fc-4bbd-aba0-f73fb0159317/8a29748a-6c5e-4612-a419-da14a8346273"
+      (reference "C127") (unit 1) (value "10uF") (footprint "Capacitor_SMD:C_0603_1608Metric")
+    )
+    (path "/00000000-0000-0000-0000-00006025abb3/af17f6b3-11fc-4bbd-aba0-f73fb0159317/4feacf69-9191-4ac0-bd53-ec15d13676c4"
+      (reference "C128") (unit 1) (value "10uF") (footprint "Capacitor_SMD:C_0603_1608Metric")
+    )
     (path "/00000000-0000-0000-0000-00006025abb3/00000000-0000-0000-0000-0000602a926e"
       (reference "D1") (unit 1) (value "green") (footprint "LED_SMD:LED_0603_1608Metric")
@@
       (reference "J1") (unit 1) (value "Conn_02x06_Odd_Even") (footprint "Connector_PinSocket_2.54mm:PinSocket_2x06_P2.54mm_Horizontal")
     )
-    (path "/00000000-0000-0000-0000-00006025abb3/00000000-0000-0000-0000-00006038cd42"
-      (reference "J2") (unit 1) (value "Conn_01x06_Male") (footprint "Connector_JST:JST_PH_S6B-PH-K_1x06_P2.00mm_Horizontal")
+    (path "/00000000-0000-0000-0000-00006025abb3/7c37e9b3-6c31-4db6-97b1-0df5756e818f"
+      (reference "J2") (unit 1) (value "Micro_SD_Card") (footprint "my_library:TF-01A")
     )
     (path "/00000000-0000-0000-0000-00006025abb3/7199a232-73f6-41ba-9a7f-9b313f9260ad"
@@
     )
     (path "/ee089113-0d86-41d6-9b05-f26d70f5fa35"
-      (reference "J5") (unit 1) (value "Conn_01x04") (footprint "Connector_PinHeader_2.54mm:PinHeader_1x04_P2.54mm_Vertical")
+      (reference "J5") (unit 1) (value "Conn_01x04") (footprint "Connector_PinSocket_2.54mm:PinSocket_1x04_P2.54mm_Vertical")
     )
     (path "/a2c655aa-ac6e-4e1c-b896-87a864540bb4"
-      (reference "J6") (unit 1) (value "Conn_01x04") (footprint "Connector_PinHeader_2.54mm:PinHeader_1x04_P2.54mm_Vertical")
+      (reference "J6") (unit 1) (value "Conn_01x04") (footprint "Connector_PinSocket_2.54mm:PinSocket_1x04_P2.54mm_Vertical")
     )
     (path "/2f24831d-7b96-4388-9dca-f54825341715"
-      (reference "J7") (unit 1) (value "Conn_01x08") (footprint "Connector_PinSocket_2.54mm:PinSocket_1x08_P2.54mm_Vertical")
+      (reference "J7") (unit 1) (value "Conn_01x08") (footprint "Connector_PinHeader_2.54mm:PinHeader_1x08_P2.54mm_Vertical")
     )
     (path "/00000000-0000-0000-0000-00006025abb3/af17f6b3-11fc-4bbd-aba0-f73fb0159317/f4b6a2da-b881-4d1c-a74c-8a240364b607"
@@
       (reference "R32") (unit 1) (value "10k") (footprint "Resistor_SMD:R_0402_1005Metric")
     )
+    (path "/00000000-0000-0000-0000-00006025abb3/d81fa49f-0176-4563-8dea-40c4bac83082"
+      (reference "R33") (unit 1) (value "10k") (footprint "Resistor_SMD:R_0402_1005Metric")
+    )
+    (path "/00000000-0000-0000-0000-00006025abb3/b73128b7-7cea-41fb-b14f-3f988c209447"
+      (reference "R34") (unit 1) (value "10k") (footprint "Resistor_SMD:R_0402_1005Metric")
+    )
+    (path "/00000000-0000-0000-0000-00006025abb3/4ccddb6d-b483-43f1-9fc3-65f55b483bfb"
+      (reference "R35") (unit 1) (value "10k") (footprint "Resistor_SMD:R_0402_1005Metric")
+    )
+    (path "/00000000-0000-0000-0000-00006025abb3/06be18ca-e7fd-42db-83ff-34e4193af719"
+      (reference "R36") (unit 1) (value "10k") (footprint "Resistor_SMD:R_0402_1005Metric")
+    )
     (path "/00000000-0000-0000-0000-00006025abb3/af17f6b3-11fc-4bbd-aba0-f73fb0159317/4885591a-d886-4219-b4c8-9ab2478f4568"

Commit message: RH v2 version
Parts:
- J10, J9: JLCPCB_CORRECTION (none) -> 0;3.81;90; LCSC (none) -> C124378
- J4: LCSC (none) -> C124416
- J5, J6: LCSC (none) -> C124413
- J7: JLCPCB_CORRECTION (none) -> 0;8.89;90; LCSC (none) -> C124381
Changed lines of the file:
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@@
+      (effects (font (size 1.27 1.27)) hide)
+    )
+    (property "LCSC" "C124381" (id 4) (at 160.02 81.28 0)
+      (effects (font (size 1.27 1.27)) hide)
+    )
+    (property "JLCPCB_CORRECTION" "0;8.89;90" (id 5) (at 160.02 81.28 0)
       (effects (font (size 1.27 1.27)) hide)
     )
@@
       (effects (font (size 1.27 1.27)) hide)
     )
+    (property "LCSC" "C124378" (id 4) (at 160.02 101.6 0)
+      (effects (font (size 1.27 1.27)) hide)
+    )
+    (property "JLCPCB_CORRECTION" "0;3.81;90" (id 5) (at 160.02 101.6 0)
+      (effects (font (size 1.27 1.27)) hide)
+    )
     (pin "1")
     (pin "2")
@@
     )
     (property "Datasheet" "~" (id 3) (at 144.78 81.28 0)
+      (effects (font (size 1.27 1.27)) hide)
+    )
+    (property "LCSC" "C124416" (id 4) (at 144.78 81.28 0)
       (effects (font (size 1.27 1.27)) hide)
     )
@@
       (effects (font (size 1.27 1.27)) hide)
     )
+    (property "LCSC" "C124413" (id 4) (at 144.78 111.76 0)
+      (effects (font (size 1.27 1.27)) hide)
+    )
     (pin "1")
     (pin "2")
@@
       (effects (font (size 1.27 1.27)) hide)
     )
+    (property "LCSC" "C124413" (id 4) (at 144.78 101.6 0)
+      (effects (font (size 1.27 1.27)) hide)
+    )
     (pin "1")
     (pin "2")
@@
     )
     (property "Datasheet" "~" (id 3) (at 160.02 111.76 0)
+      (effects (font (size 1.27 1.27)) hide)
+    )
+    (property "LCSC" "C124378" (id 4) (at 160.02 111.76 0)
+      (effects (font (size 1.27 1.27)) hide)
+    )
+    (property "JLCPCB_CORRECTION" "0;3.81;90" (id 5) (at 160.02 111.76 0)
       (effects (font (size 1.27 1.27)) hide)
     )
@@
     )
     (path "/00000000-0000-0000-0000-00006025abb3/00000000-0000-0000-0000-00006029e624"
-      (reference "BZ1") (unit 1) (value "Buzzer") (footprint "my_library:PIEZO")
+      (reference "BZ1") (unit 1) (value "Buzzer") (footprint "Robotarna_KiCad_Library:ELKS-PIEZO")
     )
     (path "/00000000-0000-0000-0000-00006025abb3/53385de2-e658-4d09-8e95-db18a23c9cb6"
@@
       (reference "J12") (unit 1) (value "Conn_01x02") (footprint "Connector_PinSocket_2.54mm:PinSocket_1x02_P2.54mm_Vertical")
     )
+    (path "/00000000-0000-0000-0000-00006025abb3/fe1b4753-aaf8-43e2-812e-ce02e6b4ce08"
+      (reference "J13") (unit 1) (value "Conn_01x03") (footprint "Connector_PinHeader_2.54mm:PinHeader_1x03_P2.54mm_Horizontal")
+    )
     (path "/00000000-0000-0000-0000-00006025abb3/af17f6b3-11fc-4bbd-aba0-f73fb0159317/d55684ea-749a-4af5-9674-faca55edf677"
       (reference "Q1") (unit 1) (value "Q_NPN_BEC") (footprint "Package_TO_SOT_SMD:SOT-23")
@@
       (reference "Q3") (unit 1) (value "Q_Photo_NPN") (footprint "my_library:SMD,3.5x2.8x1.9mm")
     )
-    (path "/00000000-0000-0000-0000-00006025abb3/00000000-0000-0000-0000-0000602e6458"
+    (path "/00000000-0000-0000-0000-00006025abb3/285fbfc0-72dd-4ae6-8769-07a5a22da123"
       (reference "Q4") (unit 1) (value "Q_NMOS_GSD") (footprint "Package_TO_SOT_SMD:SOT-23")
     )
-    (path "/00000000-0000-0000-0000-00006025abb3/00000000-0000-0000-0000-0000602e6450"
+    (path "/00000000-0000-0000-0000-00006025abb3/37a6cd66-8323-4442-ad9d-7eaecbfeab49"
       (reference "Q5") (unit 1) (value "Q_PMOS_GSD") (footprint "Package_TO_SOT_SMD:SOT-23")
     )
@@
       (reference "R14") (unit 1) (value "10k") (footprint "Resistor_SMD:R_0402_1005Metric")
     )
-    (path "/00000000-0000-0000-0000-00006025abb3/00000000-0000-0000-0000-0000602e642b"
+    (path "/00000000-0000-0000-0000-00006025abb3/46797cbd-4c01-45a8-ade2-a91332135490"
       (reference "R15") (unit 1) (value "100k") (footprint "Resistor_SMD:R_0402_1005Metric")
     )

Commit message: Change piezo
Parts:
- J4: JLCPCB_CORRECTION (none) -> 0;-8.89;90
- J5, J6: JLCPCB_CORRECTION (none) -> 0;-3.81;90
Changed lines of the file:
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@@
+      (effects (font (size 1.27 1.27)) hide)
+    )
+    (property "JLCPCB_CORRECTION" "0;-8.89;90" (id 5) (at 144.78 81.28 0)
       (effects (font (size 1.27 1.27)) hide)
     )
@@
       (effects (font (size 1.27 1.27)) hide)
     )
+    (property "JLCPCB_CORRECTION" "0;-3.81;90" (id 5) (at 144.78 111.76 0)
+      (effects (font (size 1.27 1.27)) hide)
+    )
     (pin "1")
     (pin "2")
@@
     )
     (property "LCSC" "C124413" (id 4) (at 144.78 101.6 0)
+      (effects (font (size 1.27 1.27)) hide)
+    )
+    (property "JLCPCB_CORRECTION" "0;-3.81;90" (id 5) (at 144.78 101.6 0)
       (effects (font (size 1.27 1.27)) hide)
     )
@@
     )
     (path "/00000000-0000-0000-0000-00006025abb3/00000000-0000-0000-0000-00006029e624"
-      (reference "BZ1") (unit 1) (value "Buzzer") (footprint "Robotarna_KiCad_Library:ELKS-PIEZO")
+      (reference "BZ1") (unit 1) (value "Buzzer") (footprint "Robotarna_KiCad_Library:PKLCS1212E-(RH-Logic_piezzo)")
     )
     (path "/00000000-0000-0000-0000-00006025abb3/53385de2-e658-4d09-8e95-db18a23c9cb6"

Commit message: Move C22 away from the SD card
Parts:
- B1, B2: footprint kikit:Board -> Robotarna_KiCad_Library:Board
Changed lines of the file:
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@@
       (effects (font (size 1.27 1.27)) (justify left))
     )
-    (property "Footprint" "kikit:Board" (at 191.77 66.675 0)
+    (property "Footprint" "Robotarna_KiCad_Library:Board" (at 191.77 66.675 0)
       (effects (font (size 1.27 1.27)) hide)
     )
@@
       (effects (font (size 1.27 1.27)) (justify left))
     )
-    (property "Footprint" "kikit:Board" (at 123.19 66.675 0)
+    (property "Footprint" "Robotarna_KiCad_Library:Board" (at 123.19 66.675 0)
       (effects (font (size 1.27 1.27)) hide)
     )
