File: hardware/v2.0/zadani_LED.kicad_sch (KiCad schematic)
At the start: 10 parts

Commit message: SD karta and factory files
Parts:
- D113, D3, D4, D5, D6: JLCPCB_CORRECTION 0;0;0 -> 0;0;90; LCSC C2761796 -> C2843785
Changed lines of the file:
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@@
       (effects (font (size 1.27 1.27)) (justify left top) hide)
     )
-    (property "LCSC" "C2761796" (id 4) (at 83.82 73.66 0)
-      (effects (font (size 1.27 1.27)) hide)
-    )
-    (property "JLCPCB_CORRECTION" "0;0;0" (id 5) (at 83.82 73.66 0)
+    (property "LCSC" "C2843785" (id 4) (at 83.82 73.66 0)
+      (effects (font (size 1.27 1.27)) hide)
+    )
+    (property "JLCPCB_CORRECTION" "0;0;90" (id 5) (at 83.82 73.66 0)
       (effects (font (size 1.27 1.27)) hide)
     )
@@
       (effects (font (size 1.27 1.27)) (justify left top) hide)
     )
-    (property "LCSC" "C2761796" (id 4) (at 116.84 73.66 0)
-      (effects (font (size 1.27 1.27)) hide)
-    )
-    (property "JLCPCB_CORRECTION" "0;0;0" (id 5) (at 116.84 73.66 0)
+    (property "LCSC" "C2843785" (id 4) (at 116.84 73.66 0)
+      (effects (font (size 1.27 1.27)) hide)
+    )
+    (property "JLCPCB_CORRECTION" "0;0;90" (id 5) (at 116.84 73.66 0)
       (effects (font (size 1.27 1.27)) hide)
     )
@@
       (effects (font (size 1.27 1.27)) (justify left top) hide)
     )
-    (property "LCSC" "C2761796" (id 4) (at 152.4 73.66 0)
-      (effects (font (size 1.27 1.27)) hide)
-    )
-    (property "JLCPCB_CORRECTION" "0;0;0" (id 5) (at 152.4 73.66 0)
+    (property "LCSC" "C2843785" (id 4) (at 152.4 73.66 0)
+      (effects (font (size 1.27 1.27)) hide)
+    )
+    (property "JLCPCB_CORRECTION" "0;0;90" (id 5) (at 152.4 73.66 0)
       (effects (font (size 1.27 1.27)) hide)
     )
@@
       (effects (font (size 1.27 1.27)) (justify left top) hide)
     )
-    (property "LCSC" "C2761796" (id 4) (at 185.42 73.66 0)
-      (effects (font (size 1.27 1.27)) hide)
-    )
-    (property "JLCPCB_CORRECTION" "0;0;0" (id 5) (at 185.42 73.66 0)
+    (property "LCSC" "C2843785" (id 4) (at 185.42 73.66 0)
+      (effects (font (size 1.27 1.27)) hide)
+    )
+    (property "JLCPCB_CORRECTION" "0;0;90" (id 5) (at 185.42 73.66 0)
       (effects (font (size 1.27 1.27)) hide)
     )
@@
       (effects (font (size 1.27 1.27)) (justify left top) hide)
     )
-    (property "LCSC" "C2761796" (id 4) (at 213.36 73.66 0)
-      (effects (font (size 1.27 1.27)) hide)
-    )
-    (property "JLCPCB_CORRECTION" "0;0;0" (id 5) (at 213.36 73.66 0)
-      (effects (font (size 1.27 1.27)) hide)
-    )
+    (property "LCSC" "C2843785" (id 4) (at 213.36 73.66 0)
+      (effects (font (size 1.27 1.27)) hide)
+    )
+    (property "JLCPCB_CORRECTION" "0;0;90" (id 5) (at 213.36 73.66 0)
+      (effects (font (size 1.27 1.27)) hide)
+    )

Commit message: Change piezo
Parts:
- D113, D3, D4, D5, D6: JLCPCB_CORRECTION 0;0;90 -> 0;0;270
Changed lines of the file:
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@@
       (effects (font (size 1.27 1.27)) hide)
     )
-    (property "JLCPCB_CORRECTION" "0;0;90" (id 5) (at 83.82 73.66 0)
+    (property "JLCPCB_CORRECTION" "0;0;270" (id 5) (at 83.82 73.66 0)
       (effects (font (size 1.27 1.27)) hide)
     )
@@
       (effects (font (size 1.27 1.27)) hide)
     )
-    (property "JLCPCB_CORRECTION" "0;0;90" (id 5) (at 116.84 73.66 0)
+    (property "JLCPCB_CORRECTION" "0;0;270" (id 5) (at 116.84 73.66 0)
       (effects (font (size 1.27 1.27)) hide)
     )
@@
       (effects (font (size 1.27 1.27)) hide)
     )
-    (property "JLCPCB_CORRECTION" "0;0;90" (id 5) (at 152.4 73.66 0)
+    (property "JLCPCB_CORRECTION" "0;0;270" (id 5) (at 152.4 73.66 0)
       (effects (font (size 1.27 1.27)) hide)
     )
@@
       (effects (font (size 1.27 1.27)) hide)
     )
-    (property "JLCPCB_CORRECTION" "0;0;90" (id 5) (at 185.42 73.66 0)
+    (property "JLCPCB_CORRECTION" "0;0;270" (id 5) (at 185.42 73.66 0)
       (effects (font (size 1.27 1.27)) hide)
     )
@@
       (effects (font (size 1.27 1.27)) hide)
     )
-    (property "JLCPCB_CORRECTION" "0;0;90" (id 5) (at 213.36 73.66 0)
+    (property "JLCPCB_CORRECTION" "0;0;270" (id 5) (at 213.36 73.66 0)
       (effects (font (size 1.27 1.27)) hide)
     )

Commit message: Move C22 away from the SD card
Parts:
- D113, D3, D4, D5, D6: LCSC C2843785 -> C2761796
Changed lines of the file:
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@@
       (effects (font (size 1.27 1.27)) (justify left top) hide)
     )
-    (property "LCSC" "C2843785" (at 83.82 73.66 0)
+    (property "LCSC" "C2761796" (at 83.82 73.66 0)
       (effects (font (size 1.27 1.27)) hide)
     )
@@
       (effects (font (size 1.27 1.27)) (justify left top) hide)
     )
-    (property "LCSC" "C2843785" (at 116.84 73.66 0)
+    (property "LCSC" "C2761796" (at 116.84 73.66 0)
       (effects (font (size 1.27 1.27)) hide)
     )
@@
       (effects (font (size 1.27 1.27)) (justify left top) hide)
     )
-    (property "LCSC" "C2843785" (at 152.4 73.66 0)
+    (property "LCSC" "C2761796" (at 152.4 73.66 0)
       (effects (font (size 1.27 1.27)) hide)
     )
@@
       (effects (font (size 1.27 1.27)) (justify left top) hide)
     )
-    (property "LCSC" "C2843785" (at 185.42 73.66 0)
+    (property "LCSC" "C2761796" (at 185.42 73.66 0)
       (effects (font (size 1.27 1.27)) hide)
     )
@@
       (effects (font (size 1.27 1.27)) (justify left top) hide)
     )
-    (property "LCSC" "C2843785" (at 213.36 73.66 0)
-      (effects (font (size 1.27 1.27)) hide)
-    )
+    (property "LCSC" "C2761796" (at 213.36 73.66 0)
+      (effects (font (size 1.27 1.27)) hide)
+    )
