File: hardware/v2.0/LEDky5.kicad_sch (KiCad schematic)
At the start: 10 parts

Commit message: SD karta and factory files
Parts:
- D12, D13, D14, D15, D16: JLCPCB_CORRECTION 0;0;0 -> 0;0;90; LCSC C2761796 -> C2843785
Changed lines of the file:
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@@
       (effects (font (size 1.27 1.27)) (justify left top) hide)
     )
-    (property "LCSC" "C2761796" (id 4) (at 71.12 92.71 0)
-      (effects (font (size 1.27 1.27)) hide)
-    )
-    (property "JLCPCB_CORRECTION" "0;0;0" (id 5) (at 71.12 92.71 0)
+    (property "LCSC" "C2843785" (id 4) (at 71.12 92.71 0)
+      (effects (font (size 1.27 1.27)) hide)
+    )
+    (property "JLCPCB_CORRECTION" "0;0;90" (id 5) (at 71.12 92.71 0)
       (effects (font (size 1.27 1.27)) hide)
     )
@@
       (effects (font (size 1.27 1.27)) (justify left top) hide)
     )
-    (property "LCSC" "C2761796" (id 4) (at 106.68 92.71 0)
-      (effects (font (size 1.27 1.27)) hide)
-    )
-    (property "JLCPCB_CORRECTION" "0;0;0" (id 5) (at 106.68 92.71 0)
+    (property "LCSC" "C2843785" (id 4) (at 106.68 92.71 0)
+      (effects (font (size 1.27 1.27)) hide)
+    )
+    (property "JLCPCB_CORRECTION" "0;0;90" (id 5) (at 106.68 92.71 0)
       (effects (font (size 1.27 1.27)) hide)
     )
@@
       (effects (font (size 1.27 1.27)) (justify left top) hide)
     )
-    (property "LCSC" "C2761796" (id 4) (at 139.7 92.71 0)
-      (effects (font (size 1.27 1.27)) hide)
-    )
-    (property "JLCPCB_CORRECTION" "0;0;0" (id 5) (at 139.7 92.71 0)
+    (property "LCSC" "C2843785" (id 4) (at 139.7 92.71 0)
+      (effects (font (size 1.27 1.27)) hide)
+    )
+    (property "JLCPCB_CORRECTION" "0;0;90" (id 5) (at 139.7 92.71 0)
       (effects (font (size 1.27 1.27)) hide)
     )
@@
       (effects (font (size 1.27 1.27)) (justify left top) hide)
     )
-    (property "LCSC" "C2761796" (id 4) (at 175.26 92.71 0)
-      (effects (font (size 1.27 1.27)) hide)
-    )
-    (property "JLCPCB_CORRECTION" "0;0;0" (id 5) (at 175.26 92.71 0)
+    (property "LCSC" "C2843785" (id 4) (at 175.26 92.71 0)
+      (effects (font (size 1.27 1.27)) hide)
+    )
+    (property "JLCPCB_CORRECTION" "0;0;90" (id 5) (at 175.26 92.71 0)
       (effects (font (size 1.27 1.27)) hide)
     )
@@
       (effects (font (size 1.27 1.27)) (justify left top) hide)
     )
-    (property "LCSC" "C2761796" (id 4) (at 207.01 92.71 0)
-      (effects (font (size 1.27 1.27)) hide)
-    )
-    (property "JLCPCB_CORRECTION" "0;0;0" (id 5) (at 207.01 92.71 0)
-      (effects (font (size 1.27 1.27)) hide)
-    )
+    (property "LCSC" "C2843785" (id 4) (at 207.01 92.71 0)
+      (effects (font (size 1.27 1.27)) hide)
+    )
+    (property "JLCPCB_CORRECTION" "0;0;90" (id 5) (at 207.01 92.71 0)
+      (effects (font (size 1.27 1.27)) hide)
+    )

Commit message: Change piezo
Parts:
- D12, D13, D14, D15, D16: JLCPCB_CORRECTION 0;0;90 -> 0;0;270
Changed lines of the file:
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@@
       (effects (font (size 1.27 1.27)) hide)
     )
-    (property "JLCPCB_CORRECTION" "0;0;90" (id 5) (at 71.12 92.71 0)
+    (property "JLCPCB_CORRECTION" "0;0;270" (id 5) (at 71.12 92.71 0)
       (effects (font (size 1.27 1.27)) hide)
     )
@@
       (effects (font (size 1.27 1.27)) hide)
     )
-    (property "JLCPCB_CORRECTION" "0;0;90" (id 5) (at 106.68 92.71 0)
+    (property "JLCPCB_CORRECTION" "0;0;270" (id 5) (at 106.68 92.71 0)
       (effects (font (size 1.27 1.27)) hide)
     )
@@
       (effects (font (size 1.27 1.27)) hide)
     )
-    (property "JLCPCB_CORRECTION" "0;0;90" (id 5) (at 139.7 92.71 0)
+    (property "JLCPCB_CORRECTION" "0;0;270" (id 5) (at 139.7 92.71 0)
       (effects (font (size 1.27 1.27)) hide)
     )
@@
       (effects (font (size 1.27 1.27)) hide)
     )
-    (property "JLCPCB_CORRECTION" "0;0;90" (id 5) (at 175.26 92.71 0)
+    (property "JLCPCB_CORRECTION" "0;0;270" (id 5) (at 175.26 92.71 0)
       (effects (font (size 1.27 1.27)) hide)
     )
@@
       (effects (font (size 1.27 1.27)) hide)
     )
-    (property "JLCPCB_CORRECTION" "0;0;90" (id 5) (at 207.01 92.71 0)
+    (property "JLCPCB_CORRECTION" "0;0;270" (id 5) (at 207.01 92.71 0)
       (effects (font (size 1.27 1.27)) hide)
     )

Commit message: Small tidy up
Parts:
- D22: renamed from D12; LCSC C2843785 -> C2761796
- D23: renamed from D13; LCSC C2843785 -> C2761796
- D24: renamed from D14; LCSC C2843785 -> C2761796
- D25: renamed from D15; LCSC C2843785 -> C2761796
- D26: renamed from D16; LCSC C2843785 -> C2761796
- renumbered C31 to C35, C32 to C36, C33 to C37, C34 to C38, C2 to C39
